Commit message: added ml

File: urdf/robot.urdf.xacro (robot description, xacro)
@@ -22,7 +22,7 @@
   <xacro:property name="box_size" value="0.05" />
   <!-- AGV Base -->
-  <xacro:property name="agv_base_height" value="0.27" />
+  <xacro:property name="agv_base_height" value="0.25" />
   <xacro:property name="agv_base_width" value="0.5" />
-  <xacro:property name="agv_base_length" value="0.66" />
+  <xacro:property name="agv_base_length" value="0.73" />
   <xacro:property name="agv_base_mass" value="500" />
   <!-- Macro for calculating inertia of cylinder -->
@@ -55,14 +55,14 @@
   <!-- WHEELS -->
   <xacro:omni_wheel_250 name="wheel_front_left" parent="agv_base_link">
-    <origin xyz="0.22 0.21 ${-agv_base_height/2}" rpy="0 0 0" />
+    <origin xyz="0.2083 0.2083 ${-agv_base_height/2}" rpy="0 0 0" />
   </xacro:omni_wheel_250>
   <xacro:omni_wheel_250 name="wheel_front_right" parent="agv_base_link">
-    <origin xyz="0.22 -0.21 ${-agv_base_height/2}" rpy="0 0 0" />
+    <origin xyz="0.2083 -0.2083 ${-agv_base_height/2}" rpy="0 0 0" />
   </xacro:omni_wheel_250>
   <xacro:omni_wheel_250 name="wheel_back_left" parent="agv_base_link">
-    <origin xyz="-0.22 0.21 ${-agv_base_height/2}" rpy="0 0 0" />
+    <origin xyz="-0.2083 0.2083 ${-agv_base_height/2}" rpy="0 0 0" />
   </xacro:omni_wheel_250>
   <xacro:omni_wheel_250 name="wheel_back_right" parent="agv_base_link">
-    <origin xyz="-0.22 -0.21 ${-agv_base_height/2}" rpy="0 0 0" />
+    <origin xyz="-0.2083 -0.2083 ${-agv_base_height/2}" rpy="0 0 0" />
   </xacro:omni_wheel_250>
   <!-- AGV_BASE_LINK -->
@@ -94,5 +94,5 @@
   <!-- AGV lidar -->
   <joint name="base_footprint_lidar_joint" type="fixed">
-    <origin xyz="0.13 -0.0015 0.9" rpy="0 0 0" />
+    <origin xyz="-0.217 0.0 0.39175" rpy="0 0 0" />
     <parent link="base_footprint"/>
     <child link="agv_lidar" />
