Commit message: updated urdf

File: urdf/omni_wheel.urdf.xacro (robot description, xacro)
@@ -1,4 +1,10 @@
 <?xml version="1.0"?>
 <robot xmlns:xacro="http://ros.org/wiki/xacro" name="mpo_500">
+  <!-- Macro for calculating inertia of cylinder -->
+  <xacro:macro name="cylinder_inertia" params="m r h">
+    <inertia  ixx="${m*(3*r*r+h*h)/12}" ixy = "0" ixz = "0"
+              iyy="${m*(3*r*r+h*h)/12}" iyz = "0"
+              izz="${m*r*r/2}" />
+  </xacro:macro>
   <xacro:macro name="omni_wheel_250" params="name parent *origin">
    <joint name="${name}_joint" type="fixed">
@@ -11,19 +17,19 @@
    <link name="${name}_link" type="wheel">
     <inertial>
-      <mass value="0.001" />
+      <mass value="2.1" />
       <origin xyz="0 0 0" rpy="0 0 0" />
-      <inertia ixx="0.0001" ixy="0" ixz="0" iyy="0.000001" iyz="0" izz="0.0001" />
+      <cylinder_inertia m="2.1" r="0.07825" h="0.085"/>
     </inertial>
     <visual>
-     <origin xyz="0 0 0" rpy="0 0 1.571" />
+     <origin xyz="0 0 0" rpy="1.570796326 0 0" />
      <geometry>
-        <mesh filename="package://ghost/meshes/MPO-500-WHEEL.STL"/>
+        <cylinder radius="0.07825" length="0.085"/>
      </geometry>
      <material name="Neobotix/Black" />
     </visual>
     <collision>
-     <origin xyz="0 0 0" rpy="1.59 0 0" />
+     <origin xyz="0 0 0" rpy="1.570796326 0 0" />
      <geometry>
-        <cylinder radius="0.12" length="0.1"/>
+        <cylinder radius="0.07825" length="0.085"/>
      </geometry>
     </collision>

File: urdf/robot.urdf.xacro (robot description, xacro)
@@ -22,14 +22,10 @@
   <xacro:property name="box_size" value="0.05" />
   <!-- AGV Base -->
-  <xacro:property name="agv_base_height" value="0.27" />
-  <xacro:property name="agv_base_width" value="0.5" />
-  <xacro:property name="agv_base_length" value="0.66" />
-  <xacro:property name="agv_base_mass" value="500" />
-  <!-- Macro for calculating inertia of cylinder -->
-  <xacro:macro name="cylinder_inertia" params="m r h">
-    <inertia  ixx="${m*(3*r*r+h*h)/12}" ixy = "0" ixz = "0"
-              iyy="${m*(3*r*r+h*h)/12}" iyz = "0"
-              izz="${m*r*r/2}" />
-  </xacro:macro>
+  <xacro:property name="agv_base_height" value="0.4" />
+  <xacro:property name="agv_base_lift" value="0.025" />
+  <xacro:property name="agv_base_width" value="0.495" />
+  <xacro:property name="agv_base_length" value="0.73" />
+  <xacro:property name="agv_base_mass" value="40" />
+  <xacro:property name="agv_wheel_height" value="0.07825" />
   <!-- Macro for calculating inertia of cube -->
   <xacro:macro name="cuboid_inertia" params="m w d h">
@@ -55,18 +51,18 @@
   <!-- WHEELS -->
   <xacro:omni_wheel_250 name="wheel_front_left" parent="agv_base_link">
-    <origin xyz="0.22 0.21 ${-agv_base_height/2}" rpy="0 0 0" />
+    <origin xyz="0.22 0.21 ${-agv_base_height/2-agv_base_lift + agv_wheel_height}" rpy="0 0 0" />
   </xacro:omni_wheel_250>
   <xacro:omni_wheel_250 name="wheel_front_right" parent="agv_base_link">
-    <origin xyz="0.22 -0.21 ${-agv_base_height/2}" rpy="0 0 0" />
+    <origin xyz="0.22 -0.21 ${-agv_base_height/2-agv_base_lift + agv_wheel_height}" rpy="0 0 0" />
   </xacro:omni_wheel_250>
   <xacro:omni_wheel_250 name="wheel_back_left" parent="agv_base_link">
-    <origin xyz="-0.22 0.21 ${-agv_base_height/2}" rpy="0 0 0" />
+    <origin xyz="-0.22 0.21 ${-agv_base_height/2-agv_base_lift + agv_wheel_height}" rpy="0 0 0" />
   </xacro:omni_wheel_250>
   <xacro:omni_wheel_250 name="wheel_back_right" parent="agv_base_link">
-    <origin xyz="-0.22 -0.21 ${-agv_base_height/2}" rpy="0 0 0" />
+    <origin xyz="-0.22 -0.21 ${-agv_base_height/2-agv_base_lift + agv_wheel_height}" rpy="0 0 0" />
   </xacro:omni_wheel_250>
   <!-- AGV_BASE_LINK -->
   <joint name="base_footprint_agv_base_joint" type="fixed">
-    <origin xyz="0 0 ${agv_base_height/2+0.13}" rpy="0 0 0" />
+    <origin xyz="0 0 ${agv_base_height/2+agv_base_lift}" rpy="0 0 0" />
     <parent link="base_footprint"/>
     <child link="agv_base_link" />
@@ -75,5 +71,5 @@
    <inertial>
      <mass value="${agv_base_mass}" />
-     <origin xyz="0 0 ${-agv_base_height/2-0.13}" />
+     <origin xyz="0 0 ${-agv_base_height/2-agv_base_lift}" />
      <cuboid_inertia m="${agv_base_mass}" d="${agv_base_length}" w="${agv_base_width}" h="${agv_base_height}" />
    </inertial>
@@ -94,5 +90,5 @@
   <!-- AGV lidar -->
   <joint name="base_footprint_lidar_joint" type="fixed">
-    <origin xyz="0.13 -0.0015 0.9" rpy="0 0 0" />
+    <origin xyz="0.13 -0.0015 0.46" rpy="0 0 0" />
     <parent link="base_footprint"/>
     <child link="agv_lidar" />
@@ -113,11 +109,11 @@
       <pose>${box_size/2} 0 0 0 0 0</pose>
       <visualize>false</visualize>
-      <update_rate>40</update_rate>
+      <update_rate>600</update_rate>
       <ray>
         <scan>
           <horizontal>
-            <samples>720</samples>
+            <samples>721</samples>
             <resolution>1</resolution>
-            <min_angle>${-M_PI}</min_angle>
+            <min_angle>-${M_PI}</min_angle>
             <max_angle>${M_PI}</max_angle>
           </horizontal>
@@ -125,5 +121,5 @@
         <range>
           <min>0.10</min>
-          <max>10.0</max>
+          <max>20.0</max>
           <resolution>0.001</resolution>
         </range>
@@ -142,5 +138,5 @@
       <odometryTopic>odom</odometryTopic>
       <robotBaseFrame>base_footprint</robotBaseFrame>
-      <odometryRate>12.0</odometryRate>
+      <odometryRate>600.0</odometryRate>
       <publishTF>true</publishTF>
     </plugin>
